File: haxmas.kicad_pcb (KiCad board)
At the start: 2 copper layers, 180.7 x 203.2 mm, 6 parts, among them SW1 SW_Push

Commit message: uwu
Routing:
- net Net-(BT1--): track 0.00 -> 24.8 mm, vias 0 -> 1
- net Net-(D1-K): track 132.8 -> 139.3 mm
Changed lines of the file:
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@@
 	)
 	(gr_arc
-		(start 121.95 53.86)
-		(mid 144.27 28.580757)
-		(end 166.59 53.86)
+		(start 121.948156 53.860228)
+		(mid 144.262645 28.5789)
+		(end 166.593661 53.845631)
 		(stroke
 			(width 0.05)
@@
 	)
 	(segment
+		(start 143.609 213.031)
+		(end 121.781 213.031)
+		(width 0.2)
+		(layer "F.Cu")
+		(net 2)
+	)
+	(segment
+		(start 144.32 212.32)
+		(end 143.609 213.031)
+		(width 0.2)
+		(layer "F.Cu")
+		(net 2)
+	)
+	(segment
+		(start 121.781 213.031)
+		(end 120.48 211.73)
+		(width 0.2)
+		(layer "F.Cu")
+		(net 2)
+	)
+	(via
+		(at 144.32 212.32)
+		(size 0.6)
+		(drill 0.3)
+		(layers "F.Cu" "B.Cu")
+		(net 2)
+	)
+	(segment
+		(start 144.3 212.34)
+		(end 144.32 212.32)
+		(width 0.2)
+		(layer "B.Cu")
+		(net 2)
+	)
+	(segment
+		(start 144.3 212.39)
+		(end 144.3 212.34)
+		(width 0.2)
+		(layer "B.Cu")
+		(net 2)
+	)
+	(segment
 		(start 144.44 187.69)
 		(end 127.82 204.31)
@@
 		(width 0.2)
 		(layer "F.Cu")
+		(net 4)
+	)
+	(segment
+		(start 120.48 207.23)
+		(end 113.98 207.23)
+		(width 0.2)
+		(layer "F.Cu")
